File: PCB/untitled.sch (EAGLE design)
At the start: 31 parts

Commit message: Add files via upload
Parts:
- renumbered JP1 to JA, JP2 to JB, JP3 to JC

Commit message: Add files via upload
Parts:
- D1, D2, D3, D4: device special:7SEG-CK -> special:7SEG-CA
Connections:
- net N$10: now also D2.CA1, D2.CA2; no longer D2.CK1, D2.CK2
- net N$11: now also D3.CA1, D3.CA2; no longer D3.CK1, D3.CK2
- net N$12: now also D4.CA1, D4.CA2; no longer D4.CK1, D4.CK2
- net N$9: now also D1.CA1, D1.CA2; no longer D1.CK1, D1.CK2
Changed lines of the file:
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@@
 </classes>
 <parts>
-<part name="D1" library="special" library_urn="urn:adsk.eagle:library:367" deviceset="7SEG-CK" device="" package3d_urn="urn:adsk.eagle:package:26668/2"/>
-<part name="D2" library="special" library_urn="urn:adsk.eagle:library:367" deviceset="7SEG-CK" device="" package3d_urn="urn:adsk.eagle:package:26668/2"/>
-<part name="D3" library="special" library_urn="urn:adsk.eagle:library:367" deviceset="7SEG-CK" device="" package3d_urn="urn:adsk.eagle:package:26668/2"/>
-<part name="D4" library="special" library_urn="urn:adsk.eagle:library:367" deviceset="7SEG-CK" device="" package3d_urn="urn:adsk.eagle:package:26668/2"/>
+<part name="D1" library="special" library_urn="urn:adsk.eagle:library:367" deviceset="7SEG-CA" device="" package3d_urn="urn:adsk.eagle:package:26668/2"/>
+<part name="D2" library="special" library_urn="urn:adsk.eagle:library:367" deviceset="7SEG-CA" device="" package3d_urn="urn:adsk.eagle:package:26668/2"/>
+<part name="D3" library="special" library_urn="urn:adsk.eagle:library:367" deviceset="7SEG-CA" device="" package3d_urn="urn:adsk.eagle:package:26668/2"/>
+<part name="D4" library="special" library_urn="urn:adsk.eagle:library:367" deviceset="7SEG-CA" device="" package3d_urn="urn:adsk.eagle:package:26668/2"/>
 <part name="LED1" library="led" library_urn="urn:adsk.eagle:library:259" deviceset="LED" device="5MM" package3d_urn="urn:adsk.eagle:package:15799/2"/>
 <part name="LED2" library="led" library_urn="urn:adsk.eagle:library:259" deviceset="LED" device="5MM" package3d_urn="urn:adsk.eagle:package:15799/2"/>
@@
 <attribute name="VALUE" x="-27.94" y="80.645" size="1.778" layer="96" rot="MR0"/>
 </instance>
-<instance part="JA" gate="-6" x="114.3" y="50.8" smashed="yes" rot="R270">
-<attribute name="NAME" x="114.3" y="52.07" size="1.778" layer="95"/>
-<attribute name="VALUE" x="114.3" y="45.085" size="1.778" layer="96"/>
-</instance>
 <instance part="JB" gate="-1" x="63.5" y="88.9" smashed="yes" rot="R270">
 <attribute name="NAME" x="63.5" y="90.17" size="1.778" layer="95"/>
@@
 <attribute name="VALUE" x="63.5" y="37.465" size="1.778" layer="96"/>
 </instance>
-<instance part="JB" gate="-3" x="124.46" y="60.96" smashed="yes" rot="R270">
-<attribute name="NAME" x="124.46" y="62.23" size="1.778" layer="95"/>
-<attribute name="VALUE" x="124.46" y="55.245" size="1.778" layer="96"/>
-</instance>
-<instance part="JB" gate="-4" x="111.76" y="22.86" smashed="yes" rot="MR270">
-<attribute name="NAME" x="111.76" y="24.13" size="1.778" layer="95" rot="MR0"/>
-<attribute name="VALUE" x="111.76" y="17.145" size="1.778" layer="96" rot="MR0"/>
-</instance>
-<instance part="JB" gate="-5" x="111.76" y="33.02" smashed="yes" rot="MR270">
-<attribute name="NAME" x="111.76" y="34.29" size="1.778" layer="95"/>
-<attribute name="VALUE" x="111.76" y="27.305" size="1.778" layer="96" rot="MR0"/>
-</instance>
-<instance part="JB" gate="-6" x="124.46" y="50.8" smashed="yes" rot="R270">
-<attribute name="NAME" x="124.46" y="52.07" size="1.778" layer="95"/>
-<attribute name="VALUE" x="124.46" y="45.085" size="1.778" layer="96"/>
-</instance>
 <instance part="R1" gate="G$1" x="50.8" y="104.14" smashed="yes">
 <attribute name="NAME" x="46.99" y="105.6386" size="1.778" layer="95"/>
@@
 <attribute name="VALUE" x="-10.16" y="-10.795" size="1.778" layer="96" rot="MR0"/>
 </instance>
-<instance part="JC" gate="-3" x="139.7" y="60.96" smashed="yes" rot="R270">
-<attribute name="NAME" x="139.7" y="62.23" size="1.778" layer="95"/>
-<attribute name="VALUE" x="139.7" y="55.245" size="1.778" layer="96"/>
-</instance>
 <instance part="JC" gate="-4" x="-10.16" y="-20.32" smashed="yes" rot="MR270">
 <attribute name="NAME" x="-10.16" y="-19.05" size="1.778" layer="95" rot="MR0"/>
 <attribute name="VALUE" x="-10.16" y="-26.035" size="1.778" layer="96" rot="MR0"/>
-</instance>
-<instance part="JC" gate="-5" x="137.16" y="30.48" smashed="yes" rot="MR270">
-<attribute name="NAME" x="137.16" y="31.75" size="1.778" layer="95" rot="MR0"/>
-<attribute name="VALUE" x="137.16" y="24.765" size="1.778" layer="96" rot="MR0"/>
-</instance>
-<instance part="JC" gate="-6" x="139.7" y="50.8" smashed="yes" rot="R270">
-<attribute name="NAME" x="139.7" y="52.07" size="1.778" layer="95"/>
-<attribute name="VALUE" x="139.7" y="45.085" size="1.778" layer="96"/>
 </instance>
 <instance part="PAD5" gate="G$1" x="43.18" y="-2.54" smashed="yes" rot="R180">
@@
 <net name="N$9" class="0">
 <segment>
-<pinref part="D1" gate="G$1" pin="CK2"/>
-<pinref part="D1" gate="G$1" pin="CK1"/>
+<pinref part="D1" gate="G$1" pin="CA2"/>
+<pinref part="D1" gate="G$1" pin="CA1"/>
 <wire x1="12.7" y1="99.06" x2="12.7" y2="101.6" width="0.1524" layer="91"/>
 <pinref part="T1" gate="G$1" pin="C"/>
@@
 <net name="N$10" class="0">
 <segment>
-<pinref part="D2" gate="G$1" pin="CK1"/>
-<pinref part="D2" gate="G$1" pin="CK2"/>
+<pinref part="D2" gate="G$1" pin="CA1"/>
+<pinref part="D2" gate="G$1" pin="CA2"/>
 <wire x1="12.7" y1="68.58" x2="12.7" y2="66.04" width="0.1524" layer="91"/>
 <pinref part="T2" gate="G$1" pin="C"/>
@@
 <net name="N$11" class="0">
 <segment>
-<pinref part="D3" gate="G$1" pin="CK1"/>
-<pinref part="D3" gate="G$1" pin="CK2"/>
+<pinref part="D3" gate="G$1" pin="CA1"/>
+<pinref part="D3" gate="G$1" pin="CA2"/>
 <wire x1="12.7" y1="48.26" x2="12.7" y2="45.72" width="0.1524" layer="91"/>
 <pinref part="T3" gate="G$1" pin="C"/>
@@
 <net name="N$12" class="0">
 <segment>
-<pinref part="D4" gate="G$1" pin="CK1"/>
-<pinref part="D4" gate="G$1" pin="CK2"/>
+<pinref part="D4" gate="G$1" pin="CA1"/>
+<pinref part="D4" gate="G$1" pin="CA2"/>
 <wire x1="12.7" y1="27.94" x2="12.7" y2="25.4" width="0.1524" layer="91"/>
 <pinref part="T4" gate="G$1" pin="C"/>

Commit message: Add files via upload
Connections:
- net N$1: now also JB-1.1; no longer JA-1.1
- net N$2: now also JB-1.2; no longer JA-1.2
- net N$23: now also JC-1.1; no longer JB-1.1
- net N$24: now also JC-1.2; no longer JB-1.2
- net N$25: now also JC-2.1; no longer JB-2.1
- net N$26: now also JC-2.2; no longer JB-2.2
- net N$27: now also JA-1.1; no longer JC-1.1
- net N$28: now also JA-1.2; no longer JC-1.2
- net N$29: now also JA-2.1; no longer JC-2.1
- net N$3: now also JB-2.2; no longer JA-2.2
- net N$30: now also JA-2.2; no longer JC-2.2
- net N$31: now also JA-4.1; no longer JC-4.1
- net N$32: now also JA-4.2; no longer JC-4.2
- net N$33: now also JB-3.1; no longer JA-3.1
- net N$34: now also JB-3.2; no longer JA-3.2
- net N$4: now also JB-2.1; no longer JA-2.1
- net N$5: now also JB-4.1; no longer JA-4.1
- net N$6: now also JB-4.2; no longer JA-4.2
- net N$7: now also JB-5.1; no longer JA-5.1
- net N$8: now also JB-5.2; no longer JA-5.2
Other:
- moved on the sheet: JA-1, JA-2, JA-4, JB-1, JB-2, JC-1, JC-2
